File: hardware/0.2/ftdi.kicad_sch (KiCad schematic)
At the start: 19 parts, among them U4 93LC46, U5 FT2232H

Commit message: update resistor values
Parts:
- R10: value 2K2 -> 1K; LCSC C163447 -> C105637; MPN RC0402JR-072K2L -> RC0402JR-071KL; MPN2 0402WGF2201TCE -> 0402WGF1001TCE
Changed lines of the file:
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@@
   (junction (at 157.48 51.435) (diameter 0.9144) (color 0 0 0 0))
   (junction (at 157.48 56.515) (diameter 0.9144) (color 0 0 0 0))
+  (no_connect (at 163.195 98.425))
+  (no_connect (at 163.195 103.505))
+  (no_connect (at 163.195 149.225))
+  (no_connect (at 163.195 78.105))
+  (no_connect (at 163.195 126.365))
+  (no_connect (at 163.195 123.825))
+  (no_connect (at 163.195 144.145))
+  (no_connect (at 163.195 164.465))
+  (no_connect (at 163.195 139.065))
+  (no_connect (at 102.235 159.385))
+  (no_connect (at 163.195 151.765))
+  (no_connect (at 163.195 154.305))
+  (no_connect (at 163.195 128.905))
+  (no_connect (at 61.595 133.35))
+  (no_connect (at 163.195 131.445))
+  (no_connect (at 163.195 83.185))
+  (no_connect (at 163.195 93.345))
+  (no_connect (at 163.195 146.685))
+  (no_connect (at 163.195 106.045))
+  (no_connect (at 163.195 95.885))
+  (no_connect (at 163.195 108.585))
+  (no_connect (at 163.195 141.605))
+  (no_connect (at 163.195 111.125))
+  (no_connect (at 163.195 133.985))
+  (no_connect (at 163.195 161.925))
   (no_connect (at 163.195 121.285))
-  (no_connect (at 102.235 159.385))
-  (no_connect (at 163.195 126.365))
-  (no_connect (at 163.195 151.765))
-  (no_connect (at 163.195 161.925))
-  (no_connect (at 163.195 128.905))
-  (no_connect (at 163.195 123.825))
-  (no_connect (at 163.195 133.985))
-  (no_connect (at 163.195 144.145))
-  (no_connect (at 163.195 149.225))
-  (no_connect (at 163.195 106.045))
   (no_connect (at 163.195 100.965))
-  (no_connect (at 163.195 141.605))
-  (no_connect (at 163.195 83.185))
-  (no_connect (at 163.195 103.505))
-  (no_connect (at 163.195 95.885))
-  (no_connect (at 163.195 111.125))
-  (no_connect (at 163.195 131.445))
-  (no_connect (at 163.195 98.425))
-  (no_connect (at 163.195 154.305))
-  (no_connect (at 61.595 133.35))
-  (no_connect (at 163.195 93.345))
-  (no_connect (at 163.195 164.465))
-  (no_connect (at 163.195 78.105))
-  (no_connect (at 163.195 146.685))
   (no_connect (at 163.195 156.845))
-  (no_connect (at 163.195 139.065))
-  (no_connect (at 163.195 108.585))
   (wire (pts (xy 39.37 135.89) (xy 39.37 136.525))
     (stroke (width 0) (type solid) (color 0 0 0 0))
@@
     (in_bom yes) (on_board yes)
     (property "Reference" "R10" (id 0) (at 73.66 146.685 90))
-    (property "Value" "2K2" (id 1) (at 73.66 144.145 90))
+    (property "Value" "1K" (id 1) (at 73.66 144.145 90))
     (property "Footprint" "Resistor_SMD:R_0402_1005Metric" (id 2) (at 73.66 142.367 90)
       (effects (font (size 1.27 1.27)) hide)
@@
       (effects (font (size 1.27 1.27)) hide)
     )
-    (property "LCSC" "C163447" (id 4) (at 73.66 144.145 0)
-      (effects (font (size 1.27 1.27)) hide)
-    )
-    (property "MPN" " RC0402JR-072K2L " (id 5) (at 73.66 144.145 0)
-      (effects (font (size 1.27 1.27)) hide)
-    )
-    (property "MPN2" "0402WGF2201TCE" (id 6) (at 73.66 144.145 0)
-      (effects (font (size 1.27 1.27)) hide)
-    )
+    (property "LCSC" "C105637" (id 4) (at 73.66 144.145 0)
+      (effects (font (size 1.27 1.27)) hide)
+    )
+    (property "MPN" "RC0402JR-071KL" (id 5) (at 73.66 144.145 0)
+      (effects (font (size 1.27 1.27)) hide)
+    )
+    (property "MPN2" "0402WGF1001TCE" (id 6) (at 73.66 144.145 0)
+      (effects (font (size 1.27 1.27)) hide)
+    )
